File: nano_sequencer.kicad_pcb (KiCad board)
At the start: 2 copper layers, 222 parts, among them J201 Conn_01x02, J202 Conn_02x03_Odd_Even, J203 Conn_01x02, J204 Conn_01x07, J401 euro_ribbon_conn, J402 Conn_01x03, J501 Conn_01x02_Pin, J502 Conn_01x02_Pin, J503 Conn_01x02_Pin, J504 Conn_01x02_Pin, J505 Conn_01x02_Pin, J506 Conn_01x02_Pin, J507 Conn_01x02_Pin, J508 Conn_01x02_Pin, J509 Conn_01x02_Pin, J510 Conn_01x02_Pin, J511 Conn_01x02_Pin, J512 Conn_01x02_Pin, J513 Conn_01x02_Pin, J514 Conn_01x02_Pin, J515 Conn_01x02_Pin, J516 Conn_01x02_Pin, J601 Conn_01x02_Pin, J602 Conn_01x02_Pin, J603 Conn_01x02_Pin, J604 Conn_01x02_Pin, J605 Conn_01x02_Pin, J606 Conn_01x02_Pin, J607 Conn_01x02_Pin, J608 Conn_01x02_Pin, J609 Conn_01x02_Pin, J610 Conn_01x02_Pin, J611 Conn_01x02_Pin, J612 Conn_01x02_Pin, J613 Conn_01x02_Pin, J614 Conn_01x02_Pin, J615 Conn_01x02_Pin, J616 Conn_01x02_Pin, SW501 SW, SW502 SW, SW503 SW, SW504 SW, SW505 SW, SW506 SW, SW507 SW, SW508 SW, SW509 SW, SW510 SW, SW511 SW, SW512 SW, SW513 SW, SW514 SW, SW515 SW, SW516 SW, SW517 SW, SW518 SW, SW519 SW_Push, SW520 SW_Push, U101 74LS125, U201 LM324, U202 74HC595, U203 74HC595, U302 TXB0108PW, U401 AMS1117-3.3, U402 AMS1117-5.0, U501 74HC165, U502 74HC165, U601 74HC595, U602 74HC595

Commit message: grouped components in board
Parts:
- added SW521: RotaryEncoder_Switch, RotaryEncoder:RotaryEncoder_Alps_EC11E-Switch_Vertical_H20mm, F.Cu at (64.1, 31.6)
- added SW522: RotaryEncoder_Switch, RotaryEncoder:RotaryEncoder_Alps_EC11E-Switch_Vertical_H20mm, F.Cu at (78.8, 31.6)
- moved R501 253.4 mm to (122.9, 21.8), turned to 0 degrees
- moved J501 249.7 mm to (123.9, 17.7), turned to 90 degrees
- moved SW501 249.5 mm to (127.5, 24.9), turned to -90 degrees
- moved D501 247.9 mm to (127.2, 21.8), turned to 180 degrees
- moved SW517 243.5 mm to (13.1, 2.07)
- moved SW518 242.6 mm to (23.2, 2.07)
- moved SW509 167.6 mm to (96.8, 24.9), turned to -90 degrees
- moved SW510 165.2 mm to (96.8, 37.6), turned to -90 degrees
- moved C401 155.7 mm to (-17.2, -24.8)
- moved C402 155.7 mm to (-17.2, -17.0)
- moved C403 155.7 mm to (-17.2, -9.12)
- moved C404 155.7 mm to (-17.2, -1.26)
- moved C405 155.7 mm to (-17.2, 6.58)
- moved C407 155.7 mm to (0.24, -4.81)
- moved C408 155.7 mm to (0.24, -1.77)
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- renumbered R606 to R605, R608 to R606, R609 to R607, R610 to R608, R611 to R609, R612 to R610, R613 to R611, R614 to R612, R616 to R613, R618 to R614, R619 to R615, R620 to R616, R605 to R617, R607 to R618, R615 to R619, R617 to R620
Routing:
- net GND: track 8.20 -> 0.00 mm
- net Net-(D602-K): track 0.00 -> 7.24 mm
- net Net-(D603-K): track 0.00 -> 7.24 mm
- net Net-(D605-K): track 0.00 -> 7.23 mm
- net Net-(D604-K): track 0.00 -> 7.22 mm
- net Net-(D602-A): track 0.00 -> 6.66 mm
- net Net-(D603-A): track 0.00 -> 6.65 mm
- net Net-(D504-A): track 0.00 -> 6.43 mm
- net Net-(D601-A): track 0.00 -> 6.41 mm
- net Net-(D505-A): track 0.00 -> 6.38 mm
- net Net-(D502-A): track 0.00 -> 6.36 mm
- net Net-(D503-A): track 0.00 -> 6.34 mm
- net Net-(SW504-B): track 0.00 -> 4.32 mm
- net Net-(SW503-B): track 0.00 -> 4.30 mm
- net Net-(SW505-B): track 0.00 -> 4.30 mm
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Other:
- board outline added: 99.1 x 99.1 mm

Commit message: routed half of inputs mess
Parts:
- C401, C402, C403, C404: footprint Capacitor_THT:CP_Radial_D6.3mm_P2.50mm -> Capacitor_THT:CP_Radial_Tantal_D4.5mm_P2.50mm
- moved C401 139.7 mm to (109.4, 34.3), turned to 180 degrees
- moved C405 131.1 mm to (108.2, 44.8), turned to -90 degrees
- moved C403 130.5 mm to (110.0, 20.3), turned to -90 degrees
- moved C402 128.2 mm to (100.1, 34.8)
- moved R521 115.5 mm to (75.7, 81.9), turned to -90 degrees
- moved U401 113.8 mm to (103.6, 23.9), turned to 90 degrees
- moved C410 113.2 mm to (107.2, 41.3)
- moved R520 112.4 mm to (64.5, 81.9), turned to -90 degrees
- moved C407 107.9 mm to (102.4, 30.1), turned to 180 degrees
- moved SW519 107.8 mm to (67.6, 80.9)
- moved SW520 107.8 mm to (72.6, 80.9)
- moved J402 106.4 mm to (95.4, 35.8), turned to 180 degrees
- moved C404 105.4 mm to (85.9, 21.0), turned to -90 degrees
- moved R518 104.2 mm to (109.2, 56.1)
- moved SW517 103.9 mm to (104.1, 52.2)
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Connections:
- C401 pad 1: Net-(U401-VI) -> +12V
- C402 pad 1: Net-(U402-VI) -> +12V
- C403 pad 1: Net-(U401-VO) -> +3.3V
- C404 pad 1: Net-(U402-VO) -> +5V
- C407 pad 1: Net-(U401-VO) -> +3.3V
- C408 pad 1: Net-(U402-VO) -> +5V
- U401 pad 2: Net-(U401-VO) -> +3.3V
- U401 pad 3: Net-(U401-VI) -> +12V
- U402 pad 2: Net-(U402-VO) -> +5V
- U402 pad 3: Net-(U402-VI) -> +12V
Routing:
- net +5V: track 61.3 -> 190.0 mm
- net Net-(D610-A): track 0.00 -> 73.0 mm, vias 0 -> 1
- net Net-(SW516-B): track 0.00 -> 72.1 mm, vias 0 -> 1
- net Net-(SW509-B): track 0.00 -> 68.3 mm, vias 0 -> 1
- net Net-(D611-A): track 0.00 -> 62.4 mm, vias 0 -> 1
- net Net-(SW515-B): track 0.00 -> 58.0 mm, vias 0 -> 1
- net +12V: track 33.4 -> 88.3 mm
- net Net-(D612-A): track 0.00 -> 52.6 mm, vias 0 -> 2
- net CLK_5v_unbuffered: track 0.00 -> 48.1 mm
- net Net-(SW514-B): track 0.00 -> 46.9 mm, vias 0 -> 1
- net A1: track 0.00 -> 46.3 mm
- net Net-(SW510-B): track 0.00 -> 45.2 mm, vias 0 -> 1
- net Net-(SW512-B): track 0.00 -> 39.7 mm
- net Net-(D613-A): track 0.00 -> 38.9 mm, vias 0 -> 1
- net -12V: track 66.0 -> 98.7 mm
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Other:
- board size 99.1 x 99.1 mm -> 113.2 x 100.6 mm

Commit message: routing spi traces (most of them) and a quarter of the input mess
Parts:
- moved JP601 7.76 mm to (131.1, 22.9)
- moved JP603 2.65 mm to (134.4, 22.9)
- moved JP602 2.29 mm to (137.6, 22.9)
Routing:
- net CLK_5v: track 0.00 -> 160.8 mm, vias 0 -> 8
- net MOSI_5v: track 0.00 -> 140.0 mm, vias 0 -> 2
- net CS_dac: track 0.00 -> 127.8 mm
- net cs_led: track 0.00 -> 124.7 mm, vias 0 -> 2
- net cs_165: track 0.00 -> 110.4 mm, vias 0 -> 2
- net output_CLK: track 0.00 -> 92.8 mm, vias 0 -> 2
- net MISO_5v_inputs: track 0.00 -> 80.6 mm, vias 0 -> 2
- net Net-(U601-QH'): track 0.00 -> 67.3 mm, vias 0 -> 2
- net Net-(D605-A): track 0.00 -> 58.6 mm, vias 0 -> 2
- net Net-(D604-A): track 0.00 -> 57.1 mm, vias 0 -> 2
- net Net-(D603-A): track 6.65 -> 45.9 mm, vias 0 -> 2
- net Net-(U501-DS): track 0.00 -> 34.1 mm, vias 0 -> 2
- net Net-(D602-A): track 6.66 -> 39.0 mm, vias 0 -> 4
- net output_cs_led: track 0.00 -> 14.3 mm
- net output_MOSI: track 0.00 -> 12.7 mm
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
Commit message: FINISHED ROUTING
Parts:
- J401: moved to B.Cu
- moved C404 24.3 mm to (110.1, 21.8)
- moved C403 23.6 mm to (86.6, 23.2), turned to 90 degrees
- moved C408 9.88 mm to (102.6, 30.0)
- moved U402 9.88 mm to (103.9, 23.8)
- moved C407 9.51 mm to (92.9, 30.0)
- moved U401 9.51 mm to (94.1, 23.8)
- moved J401 3.02 mm to (88.1, 41.7), turned to -90 degrees
- moved R301 1.07 mm to (74.7, 38.2), turned to 0 degrees
- moved D609 0.18 mm to (126.0, 20.5)
- moved R609 0.18 mm to (123.7, 20.4)
Connections:
- SW521 pad MP: (no net) -> GND
- SW521 pad S1: D5 -> D4
- SW521 pad S2: unconnected-(SW521-PadS2) -> GND
- SW522 pad MP: (no net) -> GND
- SW522 pad S1: D4 -> D5
- SW522 pad S2: unconnected-(SW522-PadS2) -> GND
Routing:
- net +5V: track 186.8 -> 641.6 mm, vias 0 -> 9
- net +12V: track 88.3 -> 197.7 mm, vias 0 -> 1
- net Net-(D609-A): track 6.63 -> 98.1 mm, vias 0 -> 3
- net Net-(D608-A): track 6.65 -> 97.7 mm
- net GND: track 0.00 -> 88.0 mm, vias 0 -> 88
- net Net-(D607-A): track 6.66 -> 87.4 mm
- net -12V: track 97.5 -> 176.6 mm, vias 0 -> 1
- net output_cs_led: track 14.3 -> 91.9 mm, vias 0 -> 2
- net Net-(D606-A): track 6.63 -> 76.0 mm
- net D5: track 0.00 -> 68.9 mm, vias 0 -> 2
- net Net-(SW501-B): track 4.30 -> 72.2 mm, vias 0 -> 2
- net CLK_5v: track 160.8 -> 226.8 mm, vias 8 -> 9
- net Net-(SW502-B): track 4.29 -> 63.1 mm, vias 0 -> 1
- net D4: track 0.00 -> 48.3 mm, vias 0 -> 2
- net A0: track 0.00 -> 46.5 mm
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- added copper zone on B.Cu, net GND
- added copper zone on F.Cu, net GND
Other:
- board size 113.2 x 100.6 mm -> 113.4 x 100.6 mm
- board text added: "3.3V"
- board text added: "5V"
- board text added: "cv"
- board text added: "dac"
- board text added: "gate"
- board text added: "led"

Commit message: added lcsc part numbers and fabrication files
Parts:
- C407, C408, C409, C501, C502, C601, C602: footprint LED_SMD:LED_0805_2012Metric_Pad1.15x1.40mm_HandSolder -> Capacitor_SMD:C_0805_2012Metric_Pad1.18x1.45mm_HandSolder
- D201: value LED_Small -> LED
- R236, R501, R502, R503, R504, R505, R506, R507, R508, R509, R510, R511, R512, R513, R514, R515, R516, R601, R602, R603, R604, R605, R606, R607, R608, R609, R610, R611, R612, R613, R614, R615, R616: value 3.3k -> 2k
Connections:
- SW521 pad MP: GND -> (no net)
- SW522 pad MP: GND -> (no net)
Other:
- board text added: "USB midi sequencer"
- board text added: "srFelipes"
